File: esp232.kicad_sch (KiCad schematic)
At the start: 13 parts, among them J1 RS232-Connector, J2 External-PWR, U1 MOUDLE-SEEEDUINO-XIAO-ESP32C3, U2 MAX3232

Commit message: updated schematic and layout
Parts:
- added H1, H2, H3, H4: MountingHole, MountingHole:MountingHole_2.5mm, symbol Mechanical:MountingHole
- added J3: Spare IO, Connector_PinHeader_1.27mm:PinHeader_2x04_P1.27mm_Vertical_SMD, symbol Connector_Generic:Conn_02x04_Top_Bottom
- C1, C2, C3, C4: footprint (none) -> Capacitor_SMD:C_0805_2012Metric_Pad1.18x1.45mm_HandSolder
- C5: value C -> 0.1uF; footprint (none) -> Capacitor_SMD:C_0805_2012Metric_Pad1.18x1.45mm_HandSolder
- D1, D2: footprint (none) -> LED_SMD:LED_0805_2012Metric_Pad1.15x1.40mm_HandSolder
- J1: footprint (none) -> Connector_IDC:IDC-Header_2x05_P2.54mm_Vertical
- J2: footprint (none) -> Connector_PinHeader_1.27mm:PinHeader_1x02_P1.27mm_Vertical
- R1, R2: footprint (none) -> Resistor_SMD:R_0805_2012Metric_Pad1.20x1.40mm_HandSolder
- U1: footprint MOUDLE14P-SMD-2.54-21X17.8MM -> xiao ESP32C3_PCB:MOUDLE14P-SMD-2.54-21X17.8MM
- U2: footprint (none) -> Package_SO:SOIC-16_3.9x9.9mm_P1.27mm
Connections:
- net +5V: now also R1.1; no longer D1.1 (K), D2.1 (K)
- net GND: now also D1.1 (K), D2.1 (K), J1.9 (Pin_9), J3.3 (Pin_3); no longer R1.2
- net RS232_CTS_OUT: now also J1.6 (Pin_6)
- net RS232_RTS_OUT: now also J1.4 (Pin_4)
- net RS232_RX_IN: now also J1.3 (Pin_3)
- net RS232_TX_OUT: now also J1.5 (Pin_5)
- net at D1.2 (A): now also R1.2; no longer R1.1
- net PA2: now reaches U1.1 (PA02_A0_D0)
- net PA2: now also J3.1 (Pin_1)
- net +3V3: now reaches U1.12 (3V3)
- net +3V3: now also J3.5 (Pin_5)
- net PA10: now reaches U1.3 (PA10_A2_D2)
- net PA10: now also J3.2 (Pin_2)
- net PA11: now reaches U1.4 (PA11_A3_D3)
- net PA11: now also J3.4 (Pin_4)
- net PA8: now reaches U1.5 (PA8_A4_D4_SDA)
- net PA8: now also J3.6 (Pin_6)
- net PA9: now reaches U1.6 (PA9_A5_D5_SCL)
- net PA9: now also J3.8 (Pin_8)
- net PA7: now reaches U1.9 (PA7_A8_D8_SCK)
- net PA7: now also J3.7 (Pin_7)
- no-connect marks 0 -> 5
Other:
- note added: "DB9 Pinout (Male) | 1 (DCD) | 2 (RXD) | 3 (TDX) | 4 (DTR) | 5 (GND) | | 6 (DSR) | 7 (RTS) | 8 (CTS) | 9 (RI) |"
- note added: "IDC Pinout (Female) | ? | 8 | 6 | 4 | 2 | | 9 | 7 | 5 | 3 | 1 |"
- note added: "IDC-DB9 Pin Mapping | IDC | DB9 | | 1 | 1 | | 3 | 2 | | 5 | 3 | | 7 | 4 | | 9 | 5 | | 2 | 6 | | 4 | 7 | | 6 | 8 | | 8 | 9 |"
- moved on the sheet: C1, C2, C3, C4, C5, D1, D2, J1, J2, R1, R2, U1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

Commit message: small layout improvements
Parts:
- J3: value Spare IO -> Spare IO Connector
Other:
- note added: "IO"
- note added: "MCU"
- note added: "MSIC"
- note added: "RS232"
- moved on the sheet: H1, H2, H3, H4, J2, J3

Commit message: fixed review comments
Changed lines of the file:
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@@
   )
   (symbol (lib_id "power:+3V3") (at 96.52 49.53 0) (unit 1)
-    (in_bom yes) (on_board yes) (dnp no) (fields_autoplaced)
+    (in_bom yes) (on_board yes) (dnp no)
     (property "Reference" "#PWR013" (at 96.52 53.34 0)
       (effects (font (size 1.27 1.27)) hide)
@@
         )
       )
-    )
-  )
-  (symbol (lib_id "power:PWR_FLAG") (at 154.94 35.56 90) (unit 1)
-    (in_bom yes) (on_board yes) (dnp no) (fields_autoplaced)
-    (property "Reference" "#FLG01" (at 153.035 35.56 0)
-      (effects (font (size 1.27 1.27)) hide)
-    )
-    (property "Value" "PWR_FLAG" (at 151.13 35.56 90)
-      (effects (font (size 1.27 1.27)) (justify left))
-    )
-    (property "Footprint" "" (at 154.94 35.56 0)
-      (effects (font (size 1.27 1.27)) hide)
-    )
-    (property "Datasheet" "~" (at 154.94 35.56 0)
-      (effects (font (size 1.27 1.27)) hide)
-    )
-    (pin "1")
-    (instances
-      (project "esp232"
-        (path "/42263837-7632-4b29-9542-a61a2119441e"
-          (reference "#FLG01") (unit 1)
-        )
-      )
